Commit message: updates

File: Universal_Robots_ROS2_Description/urdf/ur_platform.urdf.xacro (robot description, xacro)
@@ -55,5 +55,16 @@
    <link name="world" />
    <!-- create link fixed to the "world" -->
-   <link name="vineyard_base" />
+   <!-- <link name="vineyard_base" /> -->
+   <link name="vineyard_base">
+    <!-- <visual>
+        <origin xyz="0 0 0" rpy="0 0 0"/>
+        <geometry>
+         <mesh filename="package://ur_description/meshes/vineyard/grapevine_v2.stl" scale="1 1 1"/>
+        </geometry>
+        <material name="grey">
+          <color rgba="0.6 0.6 0.6 1.0"/>
+        </material>
+    </visual> -->
+   </link>
    <joint name="world_to_vineyard" type="fixed">
     <parent link="world"/>

Commit message: updates

File: Universal_Robots_ROS2_Description/urdf/ur_platform.urdf.xacro (robot description, xacro)
@@ -57,5 +57,5 @@
    <!-- <link name="vineyard_base" /> -->
    <link name="vineyard_base">
-    <!-- <visual>
+    <visual>
         <origin xyz="0 0 0" rpy="0 0 0"/>
         <geometry>
@@ -65,5 +65,5 @@
           <color rgba="0.6 0.6 0.6 1.0"/>
         </material>
-    </visual> -->
+    </visual>
    </link>
    <joint name="world_to_vineyard" type="fixed">

Commit message: updates

File: Universal_Robots_ROS2_Description/urdf/ur_platform.urdf.xacro (robot description, xacro)
@@ -67,8 +67,15 @@
     </visual>
    </link>
-   <joint name="world_to_vineyard" type="fixed">
+   <!-- <joint name="world_to_vineyard" type="fixed">
     <parent link="world"/>
     <child link="vineyard_base"/>
     <origin xyz="0.15 -0.9 0"/>
+   </joint> -->
+   <joint name="world_to_vineyard" type="prismatic">
+    <parent link="world"/>
+    <child link="vineyard_base"/>
+    <origin xyz="0.15 -0.25 0"/>
+    <axis xyz="0 1 0"/>
+    <limit lower="-1.0" upper="-0.5" effort="100" velocity="0.5"/>
    </joint>
      <!-- Platform -->
@@ -196,4 +203,27 @@
      <origin xyz="0.0 0.0 0.0" rpy="0 0 -1.5708" />          <!-- position robot in the world -->
    </xacro:ur_robot>
+  <link name="ee_link">
+    <visual>
+      <!-- Rotate so cylinder is horizontal -->
+      <origin xyz="0 0 -0.1" rpy="0 0 0"/>  <!-- 90° around Y -->
+      <geometry>
+        <cylinder length="0.2" radius="0.02"/>
+      </geometry>
+      <material name="grey">
+          <color rgba="0.6 0.6 0.6 1.0"/>
+        </material>
+    </visual>
+    <collision>
+      <origin xyz="0 0 -0.1" rpy="0 0 0"/>
+      <geometry>
+        <cylinder length="0.2" radius="0.02"/>
+      </geometry>
+    </collision>
+  </link>
+  <joint name="ee_joint" type="fixed">
+    <origin xyz="0 0 0.2" rpy="0 0 0"/>
+    <parent link="tool0"/>
+    <child link="ee_link"/>
+  </joint>
    <xacro:if value="$(arg sim_gazebo)">
     <!-- Gazebo plugins -->

File: Universal_Robots_ROS2_Driver/ur_moveit_config/srdf/ur_platform_macro.srdf.xacro (robot description, xacro)
@@ -12,5 +12,5 @@
     <!--SUBGROUPS - Groups can also be formed by referencing to already defined group names-->
     <group name="${prefix}${name}_manipulator">
-      <chain base_link="${prefix}base_link" tip_link="${prefix}tool0" />
+      <chain base_link="${prefix}base_link" tip_link="${prefix}ee_link" />
     </group>
     <!--GROUP STATES - Purpose - Define a named state for a particular group, in terms of joint values. This is useful to define states like 'folded arms'-->
@@ -81,4 +81,11 @@
     <disable_collisions link1="${prefix}platform_link" link2="${prefix}mount_cylinder" reason="Adjacent" />
     <disable_collisions link1="${prefix}platform_link" link2="${prefix}ground_plane" reason="Adjacent" />
+    <disable_collisions link1="${prefix}ee_link" link2="${prefix}tool0" reason="Adjacent" />
+    <disable_collisions link1="${prefix}ee_link" link2="${prefix}wrist_1_link" reason="Adjacent" />
+    <disable_collisions link1="${prefix}ee_link" link2="${prefix}wrist_2_link" reason="Adjacent" />
+    <disable_collisions link1="${prefix}ee_link" link2="${prefix}wrist_3_link" reason="Adjacent" />
+    <disable_collisions link1="${prefix}base_link" link2="${prefix}platform_link" reason="Adjacent" />
+    <disable_collisions link1="${prefix}base_link_inertia" link2="${prefix}platform_link" reason="Adjacent" />
+    <disable_collisions link1="${prefix}shoulder_link" link2="${prefix}platform_link" reason="Adjacent" />
   </xacro:macro>
 </robot>

Commit message: updates

File: Universal_Robots_ROS2_Description/urdf/ur_platform.urdf.xacro (robot description, xacro)
@@ -58,5 +58,5 @@
    <link name="vineyard_base">
     <visual>
-        <origin xyz="0 0 0" rpy="0 0 0"/>
+        <origin xyz="0 0 0.15" rpy="0 0 0"/>
         <geometry>
          <mesh filename="package://ur_description/meshes/vineyard/grapevine_v2.stl" scale="1 1 1"/>

Commit message: updates

File: Universal_Robots_ROS2_Description/urdf/ur_platform.urdf.xacro (robot description, xacro)
@@ -77,5 +77,5 @@
     <origin xyz="0.15 -0.25 0"/>
     <axis xyz="0 1 0"/>
-    <limit lower="-1.0" upper="-0.5" effort="100" velocity="0.5"/>
+    <limit lower="-1.0" upper="0.0" effort="100" velocity="0.5"/>
    </joint>
      <!-- Platform -->
@@ -222,5 +222,6 @@
   </link>
   <joint name="ee_joint" type="fixed">
-    <origin xyz="0 0 0.2" rpy="0 0 0"/>
+    <!-- <origin xyz="0 0 0.2" rpy="0 0 -1.57"/> Straight tool -->
+    <origin xyz="-0.2 0 0" rpy="0 -1.57 0"/> <!--L-shape tool -->
     <parent link="tool0"/>
     <child link="ee_link"/>
