Commit message: initial_config_optimizer

File: Universal_Robots_ROS2_Description/urdf/ur_platform.urdf.xacro (robot description, xacro)
@@ -95,5 +95,6 @@
         <geometry>
         <!-- <mesh filename="$(find ur_description)/meshes/platform/left_lateral.STL" scale="1 1 1"/> -->
-         <mesh filename="package://ur_description/meshes/platform/left_lateral.STL" scale="1 1 1"/>
+        <!-- <mesh filename="package://ur_description/meshes/platform/left_lateral.STL" scale="1 1 1"/>  -->
+        <mesh filename="package://ur_description/meshes/platform/left_portico_collision_v2.STL" scale="1 1 1"/>
         </geometry>
     </collision>
@@ -129,5 +130,6 @@
     <!-- Move up/down -->
     <axis xyz="0 0 1"/>
-    <limit lower="-0.1" upper="0.3" effort="100" velocity="0.5"/>
+    <!-- <limit lower="-0.1" upper="0.3" effort="100" velocity="0.5"/> -->
+    <limit lower="-0.1" upper="0.6" effort="100" velocity="0.5"/>
   </joint>
   <joint name="platform_to_cylinder" type="revolute">
@@ -137,5 +139,6 @@
     <origin xyz="0.15 -0.25 0.0" rpy="0 0 0"/>
     <axis xyz="1 0 0"/>
-    <limit lower="-1.57" upper="1.57" effort="10" velocity="1.0"/>
+    <!-- <limit lower="-1.57" upper="1.57" effort="10" velocity="1.0"/> -->
+    <limit lower="-1.57" upper="4.71" effort="10" velocity="1.0"/>
   </joint>
    <xacro:if value="${is_sim_gazebo or is_sim_ignition}">
@@ -222,6 +225,8 @@
   </link>
   <joint name="ee_joint" type="fixed">
-    <!-- <origin xyz="0 0 0.2" rpy="0 0 -1.57"/> Straight tool -->
-    <origin xyz="-0.2 0 0" rpy="0 -1.57 0"/> <!--L-shape tool -->
+    <!-- Straight tool -->
+    <!-- <origin xyz="0 0 0.2" rpy="0 0 -1.57"/> -->
+    <!-- L-shape tool  -->
+    <origin xyz="-0.2 0 0" rpy="0 -1.57 0"/>
     <parent link="tool0"/>
     <child link="ee_link"/>

Commit message: inital config optimization

File: Universal_Robots_ROS2_Description/urdf/ur_platform.urdf.xacro (robot description, xacro)
@@ -226,7 +226,7 @@
   <joint name="ee_joint" type="fixed">
     <!-- Straight tool -->
-    <!-- <origin xyz="0 0 0.2" rpy="0 0 -1.57"/> -->
+    <origin xyz="0 0 0.2" rpy="0 0 -1.57"/>
     <!-- L-shape tool  -->
-    <origin xyz="-0.2 0 0" rpy="0 -1.57 0"/>
+    <!-- <origin xyz="-0.2 0 0" rpy="0 -1.57 0"/> -->
     <parent link="tool0"/>
     <child link="ee_link"/>

Commit message: horizontal base slider

File: Universal_Robots_ROS2_Description/urdf/ur_platform.urdf.xacro (robot description, xacro)
@@ -105,4 +105,5 @@
     <origin xyz="0 0 0.2"/>
    </joint>
+   <link name="slider_horizontal_link"/>
    <link name="slider_link"/>
    <link name="mount_cylinder">
@@ -124,8 +125,17 @@
     </collision>
   </link>
+  <joint name="horizontal_slider" type="prismatic">
+    <parent link="platform_link"/>
+    <child link="slider_horizontal_link"/>
+    <origin xyz="0 0 0.6" rpy="0 0 0"/>
+    <!-- Move up/down -->
+    <axis xyz="0 1 0"/>
+    <!-- <limit lower="-0.1" upper="0.3" effort="100" velocity="0.5"/> -->
+    <limit lower="0.0" upper="0.3" effort="100" velocity="0.5"/>
+  </joint>
   <joint name="platform_to_slider" type="prismatic">
-    <parent link="platform_link"/>
+    <parent link="slider_horizontal_link"/>
     <child link="slider_link"/>
-    <origin xyz="0 0 0.6" rpy="0 0 0"/>
+    <origin xyz="0 0 0" rpy="0 0 0"/>
     <!-- Move up/down -->
     <axis xyz="0 0 1"/>
@@ -133,4 +143,11 @@
     <limit lower="-0.1" upper="0.6" effort="100" velocity="0.5"/>
   </joint>
+  <!-- <joint name="platform_to_slider" type="prismatic">
+    <parent link="platform_link"/>
+    <child link="slider_link"/>
+    <origin xyz="0 0 0.6" rpy="0 0 0"/>
+    <axis xyz="0 0 1"/>
+    <limit lower="-0.1" upper="0.6" effort="100" velocity="0.5"/>
+  </joint> -->
   <joint name="platform_to_cylinder" type="revolute">
     <parent link="slider_link"/>
